File: Motor.kicad_sch (KiCad schematic)
At the start: 0 parts

Commit message: Finished Updating Schematics
Parts:
- added J3, J4: Screw_Terminal_01x02, symbol Connector:Screw_Terminal_01x02
- added U5: L293D, Package_DIP:DIP-16_W7.62mm, symbol Driver_Motor:L293D
Connections:
- new net +BATT: U5.16 (VCC1), U5.8 (VCC2)
- new net FAN_B: U5.7 (2A)
- new net FAN_F: U5.2 (1A)
- new net FAN_NEG: J3.1 (Pin_1), U5.6 (2Y)
- new net FAN_POS: J3.2 (Pin_2), U5.3 (1Y)
- new net FAN_PWM: U5.1 (EN1,2)
- new net GND: U5.12 (GND), U5.13 (GND), U5.4 (GND), U5.5 (GND)
- new net RUDDER_B: U5.15 (4A)
- new net RUDDER_F: U5.10 (3A)
- new net RUDDER_NEG: J4.1 (Pin_1), U5.14 (4Y)
- new net RUDDER_POS: J4.2 (Pin_2), U5.11 (3Y)
- new net RUDDER_PWM: U5.9 (EN3,4)
Other:
- removed sheet MCU
- removed sheet Motor
- removed sheet Power
- removed sheet USB
- company: Insight Wisconsin -> (none)

Commit message: Fixed PCB errors
Parts:
- removed J4: Screw_Terminal_01x02, symbol Connector:Screw_Terminal_01x02
- added J5: Screw_Terminal_01x02, TerminalBlock:TerminalBlock_Altech_AK300-2_P5.00mm, symbol Connector:Screw_Terminal_01x02
- J3: footprint (none) -> TerminalBlock:TerminalBlock_Altech_AK300-2_P5.00mm
Connections:
- net FAN_NEG: now also J5.1 (Pin_1); no longer J3.1 (Pin_1)
- net FAN_POS: now also J5.2 (Pin_2); no longer J3.2 (Pin_2)
- net RUDDER_NEG: now also J3.1 (Pin_1)
- net RUDDER_POS: now also J3.2 (Pin_2)
Changed lines of the file:
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@@
 		(dnp no)
 		(fields_autoplaced yes)
-		(property "Reference" "J3"
+		(property "Reference" "J5"
 			(at 212.09 55.8799 0)
 			(effects
@@
 			)
 		)
-		(property "Footprint" ""
+		(property "Footprint" "TerminalBlock:TerminalBlock_Altech_AK300-2_P5.00mm"
 			(at 209.55 55.88 0)
 			(effects
@@
 		(instances
 			(project ""
+				(path "/32966cbd-337b-4fa7-b66f-bfe62b1c18c3/b4bf0452-8957-43b4-857b-1edc4fb175d7"
+					(reference "J5")
+					(unit 1)
+				)
+			)
+		)
+	)
+	(symbol
+		(lib_id "Connector:Screw_Terminal_01x02")
+		(at 213.36 132.08 0)
+		(unit 1)
+		(exclude_from_sim no)
+		(in_bom yes)
+		(on_board yes)
+		(dnp no)
+		(fields_autoplaced yes)
+		(property "Reference" "J3"
+			(at 215.9 132.0799 0)
+			(effects
+				(font
+					(size 1.27 1.27)
+				)
+				(justify left)
+			)
+		)
+		(property "Value" "Screw_Terminal_01x02"
+			(at 215.9 134.6199 0)
+			(effects
+				(font
+					(size 1.27 1.27)
+				)
+				(justify left)
+			)
+		)
+		(property "Footprint" "TerminalBlock:TerminalBlock_Altech_AK300-2_P5.00mm"
+			(at 213.36 132.08 0)
+			(effects
+				(font
+					(size 1.27 1.27)
+				)
+				(hide yes)
+			)
+		)
+		(property "Datasheet" "~"
+			(at 213.36 132.08 0)
+			(effects
+				(font
+					(size 1.27 1.27)
+				)
+				(hide yes)
+			)
+		)
+		(property "Description" "Generic screw terminal, single row, 01x02, script generated (kicad-library-utils/schlib/autogen/connector/)"
+			(at 213.36 132.08 0)
+			(effects
+				(font
+					(size 1.27 1.27)
+				)
+				(hide yes)
+			)
+		)
+		(pin "1"
+		)
+		(pin "2"
+		)
+		(instances
+			(project "Airboat"
 				(path "/32966cbd-337b-4fa7-b66f-bfe62b1c18c3/b4bf0452-8957-43b4-857b-1edc4fb175d7"
 					(reference "J3")
@@
 					(unit 1)
 				)
-			)
-		)
-	)
-	(symbol
-		(lib_id "Connector:Screw_Terminal_01x02")
-		(at 213.36 132.08 0)
-		(unit 1)
-		(exclude_from_sim no)
-		(in_bom yes)
-		(on_board yes)
-		(dnp no)
-		(fields_autoplaced yes)
-		(property "Reference" "J4"
-			(at 215.9 132.0799 0)
-			(effects
-				(font
-					(size 1.27 1.27)
-				)
-				(justify left)
-			)
-		)
-		(property "Value" "Screw_Terminal_01x02"
-			(at 215.9 134.6199 0)
-			(effects
-				(font
-					(size 1.27 1.27)
-				)
-				(justify left)
-			)
-		)
-		(property "Footprint" ""
-			(at 213.36 132.08 0)
-			(effects
-				(font
-					(size 1.27 1.27)
-				)
-				(hide yes)
-			)
-		)
-		(property "Datasheet" "~"
-			(at 213.36 132.08 0)
-			(effects
-				(font
-					(size 1.27 1.27)
-				)
-				(hide yes)
-			)
-		)
-		(property "Description" "Generic screw terminal, single row, 01x02, script generated (kicad-library-utils/schlib/autogen/connector/)"
-			(at 213.36 132.08 0)
-			(effects
-				(font
-					(size 1.27 1.27)
-				)
-				(hide yes)
-			)
-		)
-		(pin "1"
-		)
-		(pin "2"
-		)
-		(instances
-			(project "Airboat"
-				(path "/32966cbd-337b-4fa7-b66f-bfe62b1c18c3/b4bf0452-8957-43b4-857b-1edc4fb175d7"
-					(reference "J4")
-					(unit 1)
-				)
